File: hardware/board/inputs.kicad_sch (KiCad schematic)
At the start: 10 parts, among them J3 Left, J4 Right, U3 TL074

Commit message: Hardware v10:
- Replaced EOL 5V DC-DC converter with new TI part.
- Re-drawn schematic to current Winterbloom standards and style.
- Improved layout and color-coding.
- Updated branding and silk screen.
Parts:
- C18, C19: LCSC (none) -> C1653; MPN (none) -> CL10C220JB8NNNC; Notes Bulk cap -> Audio path; Rating 25V/10%/X7R -> 50V/5%/C0G
- J3, J4: mpn WQP-WQP518MA -> (none)
- R1, R5: DigiKey YAG2323TR-ND -> (none); LCSC C375503 -> C728638; MPN RT0603FRE071KL -> RT0603FRE07100KL
- R2, R6: DigiKey YAG2323TR-ND -> (none); LCSC C375503 -> C863737; MPN RT0603FRE071KL -> RT0603FRE0730KL
- RV1: MPN (none) -> Thonk 9mm B10k DUAL GANG; mpn Thonk 9mm B10k DUAL GANG -> (none)
- U3: value TL074 -> TL074H; Substitutes Allowed (none) -> No; mpn TL074CPW -> (none); populate 1 -> (none)
Changed lines of the file:
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@@
 	(title_block
 		(title "Speak to Me")
-		(date "2024-07-21")
-		(rev "v9")
+		(date "2024-08-28")
+		(rev "v10")
 		(company "Winterbloom")
 		(comment 1 "Alethea Flowers")
@@
 			)
 		)
-		(property "Notes" "Bulk cap"
+		(property "Notes" "Audio path"
 			(at 137.16 64.77 0)
 			(effects
@@
 			)
 		)
-		(property "Rating" "25V/10%/X7R"
+		(property "Rating" "50V/5%/C0G"
 			(at 137.1663 60.96 90)
 			(effects
@@
 			)
 		)
-		(property "MPN" ""
+		(property "MPN" "CL10C220JB8NNNC"
 			(at 137.16 64.77 0)
 			(effects
@@
 			)
 		)
-		(property "LCSC" ""
+		(property "LCSC" "C1653"
 			(at 137.16 64.77 0)
 			(effects
@@
 		)
 		(property "Substitutes Allowed" "Yes"
-			(at 137.16 64.77 0)
-			(effects
-				(font
-					(size 1.27 1.27)
-				)
-				(hide yes)
-			)
-		)
-		(property "search link" ""
 			(at 137.16 64.77 0)
 			(effects
@@
 			)
 		)
-		(property "Value" "TL074"
+		(property "Value" "TL074H"
 			(at 138.43 90.805 0)
 			(effects
@@
 			)
 		)
-		(property "mpn" "TL074CPW"
-			(at 137.16 93.98 0)
-			(effects
-				(font
-					(size 1.27 1.27)
-				)
-				(hide yes)
-			)
-		)
-		(property "populate" "1"
-			(at 137.16 86.36 0)
-			(effects
-				(font
-					(size 1.27 1.27)
-				)
-				(hide yes)
-			)
-		)
 		(property "Rating" ""
 			(at 137.16 86.36 0)
@@
 			)
 		)
-		(property "search link" ""
+		(property "Substitutes Allowed" "No"
 			(at 137.16 86.36 0)
 			(effects
@@
 			)
 		)
-		(property "DigiKey" "YAG2323TR-ND"
+		(property "DigiKey" ""
 			(at 119.38 83.82 0)
 			(effects
@@
 			)
 		)
-		(property "LCSC" "C375503"
+		(property "LCSC" "C728638"
 			(at 119.38 83.82 0)
 			(effects
@@
 			)
 		)
-		(property "MPN" "RT0603FRE071KL"
-			(at 119.38 83.82 0)
-			(effects
-				(font
-					(size 1.27 1.27)
-				)
-				(hide yes)
-			)
-		)
-		(property "search link" ""
+		(property "MPN" "RT0603FRE07100KL"
 			(at 119.38 83.82 0)
 			(effects
@@
 			)
 		)
-		(property "Notes" "Bulk cap"
+		(property "Notes" "Audio path"
 			(at 137.16 128.27 0)
 			(effects
@@
 			)
 		)
-		(property "Rating" "25V/10%/X7R"
+		(property "Rating" "50V/5%/C0G"
 			(at 137.1663 124.46 90)
 			(effects
@@
 			)
 		)
-		(property "MPN" ""
+		(property "MPN" "CL10C220JB8NNNC"
 			(at 137.16 128.27 0)
 			(effects
@@
 			)
 		)
-		(property "LCSC" ""
+		(property "LCSC" "C1653"
 			(at 137.16 128.27 0)
 			(effects
@@
 		)
 		(property "Substitutes Allowed" "Yes"
-			(at 137.16 128.27 0)
-			(effects
-				(font
-					(size 1.27 1.27)
-				)
-				(hide yes)
-			)
-		)
-		(property "search link" ""
 			(at 137.16 128.27 0)
 			(effects
@@
 			)
 		)
-		(property "DigiKey" "YAG2323TR-ND"
+		(property "DigiKey" ""
 			(at 119.38 147.32 0)
 			(effects
@@
 			)
 		)
-		(property "LCSC" "C375503"
+		(property "LCSC" "C728638"
 			(at 119.38 147.32 0)
 			(effects
@@
 			)
 		)
-		(property "MPN" "RT0603FRE071KL"
-			(at 119.38 147.32 0)
-			(effects
-				(font
-					(size 1.27 1.27)
-				)
-				(hide yes)
-			)
-		)
-		(property "search link" ""
+		(property "MPN" "RT0603FRE07100KL"
 			(at 119.38 147.32 0)
 			(effects
@@
 			)
 		)
-		(property "mpn" "Thonk 9mm B10k DUAL GANG"
-			(at 162.56 90.17 0)
-			(effects
-				(font
-					(size 1.27 1.27)
-				)
-				(hide yes)
-			)
-		)
-		(property "notes" ""
-			(at 162.56 90.17 0)
-			(effects
-				(font
-					(size 1.27 1.27)
-				)
-				(hide yes)
-			)
-		)
-		(property "search link" ""
+		(property "MPN" "Thonk 9mm B10k DUAL GANG"
 			(at 162.56 90.17 0)
 			(effects
@@
 			)
 		)
-		(property "mpn" "WQP-WQP518MA"
-			(at 101.6 142.24 0)
-			(effects
-				(font
-					(size 1.27 1.27)
-				)
-				(hide yes)
-			)
-		)
-		(property "search link" ""
-			(at 101.6 148.59 0)
-			(effects
-				(font
-					(size 1.27 1.27)
-				)
-				(hide yes)
-			)
-		)
 		(property "MPN" "WQP-WQP518MA"
 			(at 101.6 142.24 0)
@@
 		)
 		(property "Description" "Eurorack vertical jack, 2 Poles (Mono / TS), Switched T Pole (Normalling)"
-			(at 101.6 85.09 0)
-			(effects
-				(font
-					(size 1.27 1.27)
-				)
-				(hide yes)
-			)
-		)
-		(property "mpn" "WQP-WQP518MA"
-			(at 101.6 78.74 0)
-			(effects
-				(font
-					(size 1.27 1.27)
-				)
-				(hide yes)
-			)
-		)
-		(property "search link" ""
 			(at 101.6 85.09 0)
 			(effects
@@
 			)
 		)
-		(property "Value" "TL074"
+		(property "Value" "TL074H"
 			(at 140.335 154.305 0)
 			(effects
@@
 			)
 		)
-		(property "mpn" "TL074CPW"
-			(at 137.16 149.86 0)
-			(effects
-				(font
-					(size 1.27 1.27)
-				)
-				(hide yes)
-			)
-		)
-		(property "populate" "1"
-			(at 137.16 149.86 0)
-			(effects
-				(font
-					(size 1.27 1.27)
-				)
-				(hide yes)
-			)
-		)
 		(property "Rating" ""
 			(at 137.16 149.86 0)
@@
 			)
 		)
-		(property "search link" ""
+		(property "Substitutes Allowed" "No"
 			(at 137.16 149.86 0)
 			(effects
@@
 			)
 		)
-		(property "DigiKey" "YAG2323TR-ND"
+		(property "DigiKey" ""
 			(at 137.16 140.97 0)
 			(effects
@@
 			)
 		)
-		(property "LCSC" "C375503"
+		(property "LCSC" "C863737"
 			(at 137.16 140.97 0)
 			(effects
@@
 			)
 		)
-		(property "MPN" "RT0603FRE071KL"
-			(at 137.16 140.97 0)
-			(effects
-				(font
-					(size 1.27 1.27)
-				)
-				(hide yes)
-			)
-		)
-		(property "search link" ""
+		(property "MPN" "RT0603FRE0730KL"
 			(at 137.16 140.97 0)
 			(effects
@@
 			)
 		)
-		(property "mpn" "Thonk 9mm B10k DUAL GANG"
-			(at 163.83 153.67 0)
-			(effects
-				(font
-					(size 1.27 1.27)
-				)
-				(hide yes)
-			)
-		)
-		(property "notes" ""
-			(at 163.83 153.67 0)
-			(effects
-				(font
-					(size 1.27 1.27)
-				)
-				(hide yes)
-			)
-		)
-		(property "search link" ""
+		(property "MPN" "Thonk 9mm B10k DUAL GANG"
 			(at 163.83 153.67 0)
 			(effects
@@
 			)
 		)
-		(property "DigiKey" "YAG2323TR-ND"
+		(property "DigiKey" ""
 			(at 137.16 77.47 0)
 			(effects
@@
 			)
 		)
-		(property "LCSC" "C375503"
+		(property "LCSC" "C863737"
 			(at 137.16 77.47 0)
 			(effects
@@
 			)
 		)
-		(property "MPN" "RT0603FRE071KL"
+		(property "MPN" "RT0603FRE0730KL"
 			(at 137.16 77.47 0)
 			(effects
-				(font
-					(size 1.27 1.27)
-				)
-				(hide yes)
-			)
-		)
-		(property "search link" ""
-			(at 137.16 77.47 0)
-			(effects
